File: custom-numpad.kicad_sch (KiCad schematic)
At the start: 26 parts, among them SW1 SW_Push, SW10 SW_Push, SW11 SW_Push, SW12 SW_Push, SW2 SW_Push, SW3 SW_Push, SW4 SW_Push, SW5 SW_Push, SW6 SW_Push, SW7 SW_Push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

Commit message: added pad connections and local footprints and schematics
Parts:
- Brd1: footprint (none) -> kbd:OLED_v2
- SW1, SW10, SW11, SW12, SW2, SW3, SW4, SW5, SW6, SW7, SW8, SW9: footprint (none) -> Button_Switch_Keyboard:SW_Cherry_MX_1.00u_PCB
Connections:
- net C-0: now also SW10.1, SW11.1, SW12.1; no longer SW4.1, SW5.1, SW9.1
- net C-1: now also SW7.1, SW9.1; no longer SW10.1, SW6.1
- net C-2: now also SW4.1, SW5.1, SW6.1; no longer SW11.1, SW12.1, SW7.1
- net at D8.2 (A): now also SW7.2; no longer SW8.2
- net at SW9.2: now also D6.2 (A); no longer D9.2 (A)
- net at D5.2 (A): now also SW10.2; no longer SW5.2
- net at SW12.2: now also D4.2 (A); no longer D12.2 (A)
- net at D10.2 (A): now also SW8.2; no longer SW10.2
- net at SW4.2: now also D7.2 (A); no longer D4.2 (A)
- net at D11.2 (A): now also SW5.2; no longer SW11.2
- net at SW6.2: now also D12.2 (A); no longer D6.2 (A)
- new net: D9.2 (A), SW11.2

Commit message: wired up pcb inserted xiao blue print
Parts:
- U1: footprint (none) -> seeed xiao:MODULE_102010388
Connections:
- net 0-VCC is gone; now on net O-VCC: U1.12 (3V3)
- net C-3: no longer names the net of U1.4 (PA11_A3_D3)
Changed lines of the file:
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@@
     )
   )
-  (global_label "0-VCC" (shape output) (at 74.295 104.14 0) (fields_autoplaced)
-    (effects (font (size 1.27 1.27)) (justify left))
-    (property "Intersheetrefs" "${INTERSHEET_REFS}" (at 83.6113 104.14 0)
+  (global_label "O-VCC" (shape output) (at 74.295 104.14 0) (fields_autoplaced)
+    (effects (font (size 1.27 1.27)) (justify left))
+    (property "Intersheetrefs" "${INTERSHEET_REFS}" (at 83.7323 104.14 0)
       (effects (font (size 1.27 1.27)) (justify left) hide)
     )
@@
     (property "Intersheetrefs" "${INTERSHEET_REFS}" (at 83.9742 100.33 0)
       (effects (font (size 1.27 1.27)) (justify left) hide)
-    )
-  )
-  (global_label "C-3" (shape input) (at 32.385 107.95 180) (fields_autoplaced)
-    (effects (font (size 1.27 1.27)) (justify right))
-    (property "Intersheetrefs" "${INTERSHEET_REFS}" (at 25.4273 107.95 0)
-      (effects (font (size 1.27 1.27)) (justify right) hide)
     )
   )
@@
       (effects (font (size 1.27 1.27)) (justify left))
     )
-    (property "Footprint" "" (at 45.085 102.87 0)
-      (effects (font (size 1.27 1.27)) hide)
-    )
+    (property "Footprint" "seeed xiao:MODULE_102010388" (at 45.085 102.87 0)
+      (effects (font (size 1.27 1.27)) hide)
+    )
